File: _restore_backup_2026-07-03T01-03-15-685/heart-pcb.kicad_pcb (KiCad board)
At the start: 2 copper layers, 100 x 100 mm, 35 parts, among them Q1 2N3904, SW1 SW_SPDT, U1 NE555P

Commit message: July 3rd -- finishing touches
Connections:
- D1 pad 1: /COL -> Net-(D1-K)
- D1 pad 2: Net-(D1-A) -> /COL
- D10 pad 1: /COL -> Net-(D10-K)
- D10 pad 2: Net-(D10-A) -> /COL
- D11 pad 1: /COL -> Net-(D11-K)
- D11 pad 2: Net-(D11-A) -> /COL
- D13 pad 1: /COL -> Net-(D13-K)
- D13 pad 2: Net-(D13-A) -> /COL
- D14 pad 1: /COL -> Net-(D14-K)
- D14 pad 2: Net-(D14-A) -> /COL
- D15 pad 1: /COL -> Net-(D15-K)
- D15 pad 2: Net-(D15-A) -> /COL
- D2 pad 1: /COL -> Net-(D2-K)
- D2 pad 2: Net-(D2-A) -> /COL
- D3 pad 1: /COL -> Net-(D3-K)
- D3 pad 2: Net-(D3-A) -> /COL
- D5 pad 1: /COL -> Net-(D5-K)
- D5 pad 2: Net-(D5-A) -> /COL
- D6 pad 1: /COL -> Net-(D6-K)
- D6 pad 2: Net-(D6-A) -> /COL
- D7 pad 1: /COL -> Net-(D7-K)
- D7 pad 2: Net-(D7-A) -> /COL
- D8 pad 1: /COL -> Net-(D8-K)
- D8 pad 2: Net-(D8-A) -> /COL
- D9 pad 1: /COL -> Net-(D9-K)
- D9 pad 2: Net-(D9-A) -> /COL
- R13 pad 2: Net-(D2-A) -> Net-(D2-K)
- R14 pad 2: Net-(D3-A) -> Net-(D3-K)
- R15 pad 2: Net-(D5-A) -> Net-(D5-K)
- R16 pad 2: Net-(D6-A) -> Net-(D6-K)
- R17 pad 2: Net-(D7-A) -> Net-(D7-K)
- R18 pad 2: Net-(D8-A) -> Net-(D8-K)
- R19 pad 2: Net-(D9-A) -> Net-(D9-K)
- R2 pad 2: Net-(D1-A) -> Net-(D1-K)
- R20 pad 2: Net-(D10-A) -> Net-(D10-K)
- R21 pad 2: Net-(D11-A) -> Net-(D11-K)
- R23 pad 2: Net-(D13-A) -> Net-(D13-K)
- R24 pad 2: Net-(D14-A) -> Net-(D14-K)
- R25 pad 2: Net-(D15-A) -> Net-(D15-K)
Routing:
- net /COL: track 239.8 -> 119.8 mm
- net VCC: track 273.3 -> 209.5 mm
- net Net-(BT1-+): track 51.7 -> 0.00 mm, vias 2 -> 0
- net Net-(U1-DISCH): track 48.8 -> 0.00 mm, vias 2 -> 0
- net Net-(D7-A): track 35.9 -> 0.00 mm
- net Net-(U1-CONT): track 35.9 -> 0.00 mm
- net Net-(U1-OUT): track 21.4 -> 0.00 mm
- net Net-(U1-THRES): track 52.6 -> 32.7 mm, vias 1 -> 0
- net Net-(D10-A): track 17.0 -> 0.00 mm, vias 1 -> 0
- net Net-(D9-A): track 16.7 -> 0.00 mm
- net Net-(D2-A): track 16.0 -> 0.00 mm
- net Net-(D1-A): track 16.0 -> 0.00 mm
- net Net-(D3-A): track 15.3 -> 0.00 mm
- net Net-(D2-K): track 0.00 -> 13.4 mm
- net GND: track 72.8 -> 63.5 mm, vias 1 -> 0
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Other:
- board text removed: "From Nick"
- board text removed: "Love ya"
