File: _restore_backup_2026-07-03T01-03-15-685/heart-pcb.kicad_sch (KiCad schematic)
At the start: 35 parts, among them Q1 2N3904, SW1 SW_SPDT, U1 NE555P

Commit message: July 3rd -- finishing touches
Connections:
- net COL: now also D1.2 (A), D10.2 (A), D11.2 (A), D13.2 (A), D14.2 (A), D15.2 (A), D2.2 (A), D3.2 (A), D5.2 (A), D6.2 (A), D7.2 (A), D8.2 (A), D9.2 (A); no longer D1.1 (K), D10.1 (K), D11.1 (K), D13.1 (K), D14.1 (K), D15.1 (K), D2.1 (K), D3.1 (K), D5.1 (K), D6.1 (K), D7.1 (K), D8.1 (K), D9.1 (K)
- net at R13.2: now also D2.1 (K); no longer D2.2 (A)
- net at R20.2: now also D10.1 (K); no longer D10.2 (A)
- net at R24.2: now also D14.1 (K); no longer D14.2 (A)
- net at R23.2: now also D13.1 (K); no longer D13.2 (A)
- net at R15.2: now also D5.1 (K); no longer D5.2 (A)
- net at R18.2: now also D8.1 (K); no longer D8.2 (A)
- net at R16.2: now also D6.1 (K); no longer D6.2 (A)
- net at R2.2: now also D1.1 (K); no longer D1.2 (A)
- net at R25.2: now also D15.1 (K); no longer D15.2 (A)
- net at R14.2: now also D3.1 (K); no longer D3.2 (A)
- net at R19.2: now also D9.1 (K); no longer D9.2 (A)
- net at R17.2: now also D7.1 (K); no longer D7.2 (A)
- net at R21.2: now also D11.1 (K); no longer D11.2 (A)
Other:
- moved on the sheet: D1, D10, D11, D13, D14, D15, D2, D3, D5, D6, D7, D8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
Changed lines of the file:
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@@
 	(symbol
 		(lib_id "Device:LED")
-		(at 220.98 139.7 180)
+		(at 220.98 139.7 0)
 		(unit 1)
 		(body_style 1)
@@
 		(fields_autoplaced yes)
 		(property "Reference" "D10"
-			(at 222.5675 132.08 0)
+			(at 219.3925 133.35 0)
 			(show_name no)
 			(do_not_autoplace no)
@@
 		)
 		(property "Value" "LED"
-			(at 222.5675 134.62 0)
+			(at 219.3925 135.89 0)
 			(show_name no)
 			(do_not_autoplace no)
@@
 	(symbol
 		(lib_id "Device:LED")
-		(at 204.47 149.86 180)
+		(at 204.47 149.86 0)
 		(unit 1)
 		(body_style 1)
@@
 		(fields_autoplaced yes)
 		(property "Reference" "D14"
-			(at 206.0575 142.24 0)
+			(at 202.8825 143.51 0)
 			(show_name no)
 			(do_not_autoplace no)
@@
 		)
 		(property "Value" "LED"
-			(at 206.0575 144.78 0)
+			(at 202.8825 146.05 0)
 			(show_name no)
 			(do_not_autoplace no)
@@
 	(symbol
 		(lib_id "Device:LED")
-		(at 180.34 152.4 180)
+		(at 180.34 152.4 0)
 		(unit 1)
 		(body_style 1)
@@
 		(fields_autoplaced yes)
 		(property "Reference" "D13"
-			(at 181.9275 144.78 0)
+			(at 178.7525 146.05 0)
 			(show_name no)
 			(do_not_autoplace no)
@@
 		)
 		(property "Value" "LED"
-			(at 181.9275 147.32 0)
+			(at 178.7525 148.59 0)
 			(show_name no)
 			(do_not_autoplace no)
@@
 	(symbol
 		(lib_id "Device:LED")
-		(at 250.19 52.07 180)
+		(at 250.19 52.07 0)
 		(unit 1)
 		(body_style 1)
@@
 		(fields_autoplaced yes)
 		(property "Reference" "D5"
-			(at 251.7775 44.45 0)
+			(at 248.6025 45.72 0)
 			(show_name no)
 			(do_not_autoplace no)
@@
 		)
 		(property "Value" "LED"
-			(at 251.7775 46.99 0)
+			(at 248.6025 48.26 0)
 			(show_name no)
 			(do_not_autoplace no)
@@
 	(symbol
 		(lib_id "Device:LED")
-		(at 146.05 114.3 180)
+		(at 146.05 114.3 0)
 		(unit 1)
 		(body_style 1)
@@
 		(fields_autoplaced yes)
 		(property "Reference" "D1"
-			(at 147.6375 106.68 0)
+			(at 144.4625 107.95 0)
 			(show_name no)
 			(do_not_autoplace no)
@@
 		)
 		(property "Value" "LED"
-			(at 147.6375 109.22 0)
+			(at 144.4625 110.49 0)
 			(show_name no)
 			(do_not_autoplace no)
@@
 	(symbol
 		(lib_id "Device:LED")
-		(at 184.15 115.57 180)
+		(at 184.15 115.57 0)
 		(unit 1)
 		(body_style 1)
@@
 		(fields_autoplaced yes)
 		(property "Reference" "D9"
-			(at 185.7375 107.95 0)
+			(at 182.5625 109.22 0)
 			(show_name no)
 			(do_not_autoplace no)
@@
 		)
 		(property "Value" "LED"
-			(at 185.7375 110.49 0)
+			(at 182.5625 111.76 0)
 			(show_name no)
 			(do_not_autoplace no)
@@
 	(symbol
 		(lib_id "Device:LED")
-		(at 146.05 158.75 180)
+		(at 146.05 158.75 0)
 		(unit 1)
 		(body_style 1)
@@
 		(fields_autoplaced yes)
 		(property "Reference" "D15"
-			(at 147.6375 151.13 0)
+			(at 144.4625 152.4 0)
 			(show_name no)
 			(do_not_autoplace no)
@@
 		)
 		(property "Value" "LED"
-			(at 147.6375 153.67 0)
+			(at 144.4625 154.94 0)
 			(show_name no)
 			(do_not_autoplace no)
@@
 	(symbol
 		(lib_id "Device:LED")
-		(at 204.47 102.87 180)
+		(at 204.47 102.87 0)
 		(unit 1)
 		(body_style 1)
@@
 		(fields_autoplaced yes)
 		(property "Reference" "D8"
-			(at 206.0575 95.25 0)
+			(at 202.8825 96.52 0)
 			(show_name no)
 			(do_not_autoplace no)
@@
 		)
 		(property "Value" "LED"
-			(at 206.0575 97.79 0)
+			(at 202.8825 99.06 0)
 			(show_name no)
 			(do_not_autoplace no)
@@
 	(symbol
 		(lib_id "Device:LED")
-		(at 207.01 67.31 180)
+		(at 207.01 67.31 0)
 		(unit 1)
 		(body_style 1)
@@
 		(fields_autoplaced yes)
 		(property "Reference" "D3"
-			(at 208.5975 59.69 0)
+			(at 205.4225 60.96 0)
 			(show_name no)
 			(do_not_autoplace no)
@@
 		)
 		(property "Value" "LED"
-			(at 208.5975 62.23 0)
+			(at 205.4225 63.5 0)
 			(show_name no)
 			(do_not_autoplace no)
@@
 	(symbol
 		(lib_id "Device:LED")
-		(at 168.91 78.74 180)
+		(at 168.91 78.74 0)
 		(unit 1)
 		(body_style 1)
@@
 		(fields_autoplaced yes)
 		(property "Reference" "D2"
-			(at 170.4975 71.12 0)
+			(at 167.3225 72.39 0)
 			(show_name no)
 			(do_not_autoplace no)
@@
 		)
 		(property "Value" "LED"
-			(at 170.4975 73.66 0)
+			(at 167.3225 74.93 0)
 			(show_name no)
 			(do_not_autoplace no)
@@
 	(symbol
 		(lib_id "Device:LED")
-		(at 224.79 105.41 180)
+		(at 224.79 105.41 0)
 		(unit 1)
 		(body_style 1)
@@
 		(fields_autoplaced yes)
 		(property "Reference" "D7"
-			(at 226.3775 97.79 0)
+			(at 223.2025 99.06 0)
 			(show_name no)
 			(do_not_autoplace no)
@@
 		)
 		(property "Value" "LED"
-			(at 226.3775 100.33 0)
+			(at 223.2025 101.6 0)
 			(show_name no)
 			(do_not_autoplace no)
@@
 	(symbol
 		(lib_id "Device:LED")
-		(at 251.46 90.17 180)
+		(at 251.46 90.17 0)
 		(unit 1)
 		(body_style 1)
@@
 		(fields_autoplaced yes)
 		(property "Reference" "D6"
-			(at 253.0475 82.55 0)
+			(at 249.8725 83.82 0)
 			(show_name no)
 			(do_not_autoplace no)
@@
 		)
 		(property "Value" "LED"
-			(at 253.0475 85.09 0)
+			(at 249.8725 86.36 0)
 			(show_name no)
 			(do_not_autoplace no)
@@
 	(symbol
 		(lib_id "Device:LED")
-		(at 259.08 137.16 180)
+		(at 259.08 137.16 0)
 		(unit 1)
 		(body_style 1)
@@
 		(fields_autoplaced yes)
 		(property "Reference" "D11"
-			(at 260.6675 129.54 0)
+			(at 257.4925 130.81 0)
 			(show_name no)
 			(do_not_autoplace no)
@@
 		)
 		(property "Value" "LED"
-			(at 260.6675 132.08 0)
+			(at 257.4925 133.35 0)
 			(show_name no)
 			(do_not_autoplace no)
